Commit message: Convert stls to objs

File: src/description/urdf/tibble_core.xacro (robot description, xacro)
@@ -26,5 +26,5 @@
       <geometry>
         <mesh
-          filename="package://description/meshes/Chassis.STL" />
+          filename="package://description/meshes/Chassis.obj" />
       </geometry>
       <material
@@ -40,5 +40,5 @@
       <geometry>
         <mesh
-          filename="package://description/meshes/Chassis.STL" />
+          filename="package://description/meshes/Chassis.obj" />
       </geometry>
     </collision>
@@ -77,5 +77,5 @@
       <geometry>
         <mesh
-          filename="package://description/meshes/DL_Wheel.STL" />
+          filename="package://description/meshes/DL_Wheel.obj" />
       </geometry>
       <material
@@ -91,5 +91,5 @@
       <geometry>
         <mesh
-          filename="package://description/meshes/DL_Wheel.STL" />
+          filename="package://description/meshes/DL_Wheel.obj" />
       </geometry>
     </collision>
@@ -130,19 +130,19 @@
       <geometry>
         <mesh
-          filename="package://description/meshes/DR_Wheel.STL" />
-      </geometry>
-      <material
-        name="">
-        <color
-          rgba="0.792156862745098 0.819607843137255 0.933333333333333 1" />
-      </material>
-    </visual>
-    <collision>
-      <origin
-        xyz="0 0 0"
-        rpy="0 0 0" />
-      <geometry>
-        <mesh
-          filename="package://description/meshes/DR_Wheel.STL" />
+          filename="package://description/meshes/DR_Wheel.obj" />
+      </geometry>
+      <material
+        name="">
+        <color
+          rgba="0.792156862745098 0.819607843137255 0.933333333333333 1" />
+      </material>
+    </visual>
+    <collision>
+      <origin
+        xyz="0 0 0"
+        rpy="0 0 0" />
+      <geometry>
+        <mesh
+          filename="package://description/meshes/DR_Wheel.obj" />
       </geometry>
     </collision>
@@ -183,19 +183,19 @@
       <geometry>
         <mesh
-          filename="package://description/meshes/BLA.STL" />
-      </geometry>
-      <material
-        name="">
-        <color
-          rgba="0.792156862745098 0.819607843137255 0.933333333333333 1" />
-      </material>
-    </visual>
-    <collision>
-      <origin
-        xyz="0 0 0"
-        rpy="0 0 0" />
-      <geometry>
-        <mesh
-          filename="package://description/meshes/BLA.STL" />
+          filename="package://description/meshes/BLA.obj" />
+      </geometry>
+      <material
+        name="">
+        <color
+          rgba="0.792156862745098 0.819607843137255 0.933333333333333 1" />
+      </material>
+    </visual>
+    <collision>
+      <origin
+        xyz="0 0 0"
+        rpy="0 0 0" />
+      <geometry>
+        <mesh
+          filename="package://description/meshes/BLA.obj" />
       </geometry>
     </collision>
@@ -241,19 +241,19 @@
       <geometry>
         <mesh
-          filename="package://description/meshes/LA.STL" />
-      </geometry>
-      <material
-        name="">
-        <color
-          rgba="0.792156862745098 0.819607843137255 0.933333333333333 1" />
-      </material>
-    </visual>
-    <collision>
-      <origin
-        xyz="0 0 0"
-        rpy="0 0 0" />
-      <geometry>
-        <mesh
-          filename="package://description/meshes/LA.STL" />
+          filename="package://description/meshes/LA.obj" />
+      </geometry>
+      <material
+        name="">
+        <color
+          rgba="0.792156862745098 0.819607843137255 0.933333333333333 1" />
+      </material>
+    </visual>
+    <collision>
+      <origin
+        xyz="0 0 0"
+        rpy="0 0 0" />
+      <geometry>
+        <mesh
+          filename="package://description/meshes/LA.obj" />
       </geometry>
     </collision>
@@ -299,19 +299,19 @@
       <geometry>
         <mesh
-          filename="package://description/meshes/TLA.STL" />
-      </geometry>
-      <material
-        name="">
-        <color
-          rgba="0.792156862745098 0.819607843137255 0.933333333333333 1" />
-      </material>
-    </visual>
-    <collision>
-      <origin
-        xyz="0 0 0"
-        rpy="0 0 0" />
-      <geometry>
-        <mesh
-          filename="package://description/meshes/TLA.STL" />
+          filename="package://description/meshes/TLA.obj" />
+      </geometry>
+      <material
+        name="">
+        <color
+          rgba="0.792156862745098 0.819607843137255 0.933333333333333 1" />
+      </material>
+    </visual>
+    <collision>
+      <origin
+        xyz="0 0 0"
+        rpy="0 0 0" />
+      <geometry>
+        <mesh
+          filename="package://description/meshes/TLA.obj" />
       </geometry>
     </collision>
@@ -357,5 +357,5 @@
       <geometry>
         <mesh
-          filename="package://description/meshes/Hopper.STL" />
+          filename="package://description/meshes/Hopper.obj" />
       </geometry>
       <material
@@ -371,5 +371,5 @@
       <geometry>
         <mesh
-          filename="package://description/meshes/Hopper.STL" />
+          filename="package://description/meshes/Hopper.obj" />
       </geometry>
     </collision>
@@ -415,5 +415,5 @@
       <geometry>
         <mesh
-          filename="package://description/meshes/Hopper_Door.STL" />
+          filename="package://description/meshes/Hopper_Door.obj" />
       </geometry>
       <material
@@ -429,5 +429,5 @@
       <geometry>
         <mesh
-          filename="package://description/meshes/Hopper_Door.STL" />
+          filename="package://description/meshes/Hopper_Door.obj" />
       </geometry>
     </collision>
@@ -473,5 +473,5 @@
       <geometry>
         <mesh
-          filename="package://description/meshes/Hopper_Latch.STL" />
+          filename="package://description/meshes/Hopper_Latch.obj" />
       </geometry>
       <material
@@ -487,5 +487,5 @@
       <geometry>
         <mesh
-          filename="package://description/meshes/Hopper_Latch.STL" />
+          filename="package://description/meshes/Hopper_Latch.obj" />
       </geometry>
     </collision>
@@ -531,19 +531,19 @@
       <geometry>
         <mesh
-          filename="package://description/meshes/Excavation.STL" />
-      </geometry>
-      <material
-        name="">
-        <color
-          rgba="0.792156862745098 0.819607843137255 0.933333333333333 1" />
-      </material>
-    </visual>
-    <collision>
-      <origin
-        xyz="0 0 0"
-        rpy="0 0 0" />
-      <geometry>
-        <mesh
-          filename="package://description/meshes/Excavation.STL" />
+          filename="package://description/meshes/Excavation.obj" />
+      </geometry>
+      <material
+        name="">
+        <color
+          rgba="0.792156862745098 0.819607843137255 0.933333333333333 1" />
+      </material>
+    </visual>
+    <collision>
+      <origin
+        xyz="0 0 0"
+        rpy="0 0 0" />
+      <geometry>
+        <mesh
+          filename="package://description/meshes/Excavation.obj" />
       </geometry>
     </collision>
@@ -584,19 +584,19 @@
       <geometry>
         <mesh
-          filename="package://description/meshes/FL_Wheel.STL" />
-      </geometry>
-      <material
-        name="">
-        <color
-          rgba="0.792156862745098 0.819607843137255 0.933333333333333 1" />
-      </material>
-    </visual>
-    <collision>
-      <origin
-        xyz="0 0 0"
-        rpy="0 0 0" />
-      <geometry>
-        <mesh
-          filename="package://description/meshes/FL_Wheel.STL" />
+          filename="package://description/meshes/FL_Wheel.obj" />
+      </geometry>
+      <material
+        name="">
+        <color
+          rgba="0.792156862745098 0.819607843137255 0.933333333333333 1" />
+      </material>
+    </visual>
+    <collision>
+      <origin
+        xyz="0 0 0"
+        rpy="0 0 0" />
+      <geometry>
+        <mesh
+          filename="package://description/meshes/FL_Wheel.obj" />
       </geometry>
     </collision>
@@ -637,19 +637,19 @@
       <geometry>
         <mesh
-          filename="package://description/meshes/ML_Wheel.STL" />
-      </geometry>
-      <material
-        name="">
-        <color
-          rgba="0.792156862745098 0.819607843137255 0.933333333333333 1" />
-      </material>
-    </visual>
-    <collision>
-      <origin
-        xyz="0 0 0"
-        rpy="0 0 0" />
-      <geometry>
-        <mesh
-          filename="package://description/meshes/ML_Wheel.STL" />
+          filename="package://description/meshes/ML_Wheel.obj" />
+      </geometry>
+      <material
+        name="">
+        <color
+          rgba="0.792156862745098 0.819607843137255 0.933333333333333 1" />
+      </material>
+    </visual>
+    <collision>
+      <origin
+        xyz="0 0 0"
+        rpy="0 0 0" />
+      <geometry>
+        <mesh
+          filename="package://description/meshes/ML_Wheel.obj" />
       </geometry>
     </collision>
@@ -690,19 +690,19 @@
       <geometry>
         <mesh
-          filename="package://description/meshes/BL_Wheel.STL" />
-      </geometry>
-      <material
-        name="">
-        <color
-          rgba="0.792156862745098 0.819607843137255 0.933333333333333 1" />
-      </material>
-    </visual>
-    <collision>
-      <origin
-        xyz="0 0 0"
-        rpy="0 0 0" />
-      <geometry>
-        <mesh
-          filename="package://description/meshes/BL_Wheel.STL" />
+          filename="package://description/meshes/BL_Wheel.obj" />
+      </geometry>
+      <material
+        name="">
+        <color
+          rgba="0.792156862745098 0.819607843137255 0.933333333333333 1" />
+      </material>
+    </visual>
+    <collision>
+      <origin
+        xyz="0 0 0"
+        rpy="0 0 0" />
+      <geometry>
+        <mesh
+          filename="package://description/meshes/BL_Wheel.obj" />
       </geometry>
     </collision>
@@ -743,19 +743,19 @@
       <geometry>
         <mesh
-          filename="package://description/meshes/TL_Wheel.STL" />
-      </geometry>
-      <material
-        name="">
-        <color
-          rgba="0.792156862745098 0.819607843137255 0.933333333333333 1" />
-      </material>
-    </visual>
-    <collision>
-      <origin
-        xyz="0 0 0"
-        rpy="0 0 0" />
-      <geometry>
-        <mesh
-          filename="package://description/meshes/TL_Wheel.STL" />
+          filename="package://description/meshes/TL_Wheel.obj" />
+      </geometry>
+      <material
+        name="">
+        <color
+          rgba="0.792156862745098 0.819607843137255 0.933333333333333 1" />
+      </material>
+    </visual>
+    <collision>
+      <origin
+        xyz="0 0 0"
+        rpy="0 0 0" />
+      <geometry>
+        <mesh
+          filename="package://description/meshes/TL_Wheel.obj" />
       </geometry>
     </collision>
@@ -796,19 +796,19 @@
       <geometry>
         <mesh
-          filename="package://description/meshes/FR_Wheel.STL" />
-      </geometry>
-      <material
-        name="">
-        <color
-          rgba="0.792156862745098 0.819607843137255 0.933333333333333 1" />
-      </material>
-    </visual>
-    <collision>
-      <origin
-        xyz="0 0 0"
-        rpy="0 0 0" />
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