Commit message: Remove sensors until we get the correct position

File: src/description/urdf/mujoco_inputs.xacro (robot description, xacro)
@@ -13,15 +13,15 @@
         </default>
       </default>
-      <actuator>
-        <velocity name="DL_Rotate" joint="DL_Rotate" kv="20"/>
-        <velocity name="RL_Rotate" joint="RL_Rotate" kv="20"/>
+      <!-- <actuator>
+        <velocity name="DL_Rotate" joint="DL_Rotate"/>
+        <velocity name="DR_Rotate" joint="DR_Rotate"/>
       </actuator>
       <actuator>
-        <velocity name="LA_Extend" joint="LA_Extend" kv="20"/>
+        <velocity name="LA_Extend" joint="LA_Extend"/>
       </actuator>
       <actuator>
         <velocity name="Excavation_Rotate" joint="Excavation_Rotate"/>
-      </actuator>
-      <extension>
+      </actuator> -->
+      <!-- <extension>
         <plugin plugin="mujoco.plugin.lidar">
           <instance name="lidar">
@@ -33,8 +33,8 @@
           </instance>
         </plugin>
-      </extension>
-      <sensor>
+      </extension> -->
+      <!-- <sensor>
         <plugin name="lidar" instance="lidar" objtype="site" objname="lidar_link_optical"/>
-      </sensor>
+      </sensor> -->
     </raw_inputs>
     <!-- Specific inputs that require processing from the conversion script-->
@@ -44,5 +44,5 @@
       <!-- The camera with the specified values will be added at the specified site name. -->
       <!-- The position and quaterinion will be filled in by the converter -->
-      <camera site="camera_link_optical" name="camera" fovy="58" mode="fixed" resolution="640 480"/>
+      <!-- <camera site="camera_link_optical" name="camera" fovy="58" mode="fixed" resolution="640 480"/> -->
       <!-- The element with the type and name as listed below will be modified with the remaining attributes -->
       <!-- If the attribute already existed, it will be overwritten -->

File: src/description/urdf/tibble.urdf.xacro (robot description, xacro)
@@ -9,5 +9,5 @@
     <!-- Include needed files (utilizing conditions) (these are relative filepaths) -->
     <xacro:include filename="tibble_core.xacro"/>
-    <xacro:include filename="sensors.xacro"/>
+    <!-- <xacro:include filename="sensors.xacro"/> -->
     <xacro:if value="$(arg use_control)">
         <xacro:include filename="ros2_control.xacro"/>

File: src/description/urdf/tibble_core.xacro (robot description, xacro)
@@ -940,12 +940,12 @@
         rpy="0 0 0" />
       <mass
-        value="0" />
-      <inertia
-        ixx="0"
-        ixy="0"
-        ixz="0"
-        iyy="0"
-        iyz="0"
-        izz="0" />
+        value="0.146434890659902" />
+      <inertia
+        ixx="8.80633224784676E-05"
+        ixy="-2.39106895777931E-22"
+        ixz="-1.34026306833892E-19"
+        iyy="8.80633224784676E-05"
+        iyz="-4.00087992203459E-19"
+        izz="0.000154471460357356" />
     </inertial>
     <visual>

Commit message: Use front wheels instead of motor wheel

File: src/description/urdf/mujoco_inputs.xacro (robot description, xacro)
@@ -14,18 +14,16 @@
       </default>
       <actuator>
-        <velocity name="DL_Rotate" joint="DL_Rotate" />
-        <velocity name="DR_Rotate" joint="DR_Rotate" />
+        <velocity name="FL_Wheel_Rotate" joint="FL_Wheel_Rotate" />
+        <velocity name="FR_Wheel_Rotate" joint="FR_Wheel_Rotate" />
         <velocity name="LA_Extend" joint="LA_Extend" />
         <velocity name="Excavation_Rotate" joint="Excavation_Rotate" />
       </actuator>
       <equality>
-        <joint joint1="FL_Wheel_Rotate" joint2="DL_Rotate"/>
-        <joint joint1="ML_Wheel_Rotate" joint2="DL_Rotate"/>
-        <joint joint1="BL_Wheel_Rotate" joint2="DL_Rotate"/>
-        <joint joint1="TL_Wheel_Rotate" joint2="DL_Rotate"/>
-        <joint joint1="FR_Wheel_Rotate" joint2="DR_Rotate"/>
-        <joint joint1="MR_Wheel_Rotate" joint2="DR_Rotate"/>
-        <joint joint1="BR_Wheel_Rotate" joint2="DR_Rotate"/>
-        <joint joint1="TR_Wheel_Rotate" joint2="DR_Rotate"/>
+        <joint joint1="ML_Wheel_Rotate" joint2="FL_Wheel_Rotate"/>
+        <joint joint1="BL_Wheel_Rotate" joint2="FL_Wheel_Rotate"/>
+        <joint joint1="TL_Wheel_Rotate" joint2="FL_Wheel_Rotate"/>
+        <joint joint1="MR_Wheel_Rotate" joint2="FR_Wheel_Rotate"/>
+        <joint joint1="BR_Wheel_Rotate" joint2="FR_Wheel_Rotate"/>
+        <joint joint1="TR_Wheel_Rotate" joint2="FR_Wheel_Rotate"/>
       </equality>
       <!-- <extension>

File: src/description/urdf/ros2_control.xacro (robot description, xacro)
@@ -66,5 +66,5 @@
             </hardware>
             <!-- Define all the joints that will have a command or state interface -->
-            <joint name="DL_Rotate">
+            <joint name="FL_Wheel_Rotate">
                 <command_interface name="velocity">
                     <param name="min">-10</param>
@@ -75,5 +75,5 @@
                 <state_interface name="velocity"/>
             </joint>
-            <joint name="DR_Rotate">
+            <joint name="FR_Wheel_Rotate">
                 <command_interface name="velocity">
                     <param name="min">-10</param>
