Commit message: Remove gazebo; add MuJoCo ROS2_Control and inputs; add dummy sensors

File: src/description/urdf/ros2_control.xacro (robot description, xacro)
@@ -60,15 +60,50 @@
     <!-- Load the ROS2 Control information for just sim purposes -->
     <xacro:if value="$(arg use_sim)">
-        <ros2_control name="name" type="system">
+        <ros2_control name="MujocoSystem" type="system">
             <hardware>
-                <plugin>gz_ros2_control/GazeboSimSystem</plugin>
+                <plugin>mujoco_ros2_control/MujocoSystemInterface</plugin>
             </hardware>
-            <!-- Define all joints and their command/state interfaces necessary for sim -->
+             <!-- Define all the joints that will have a command or state interface -->
+            <joint name="DL_Rotate">
+                <command_interface name="velocity">
+                    <param name="min">-10</param>
+                    <param name="max">10</param>
+                </command_interface>
+                <command_interface name="position"/>
+                <state_interface name="position"/>
+                <state_interface name="velocity"/>
+            </joint>
+            <joint name="DR_Rotate">
+                <command_interface name="velocity">
+                    <param name="min">-10</param>
+                    <param name="max">10</param>
+                </command_interface>
+                <command_interface name="position"/>
+                <state_interface name="position"/>
+                <state_interface name="velocity"/>
+            </joint>
+            <joint name="LA_Extend">
+                <command_interface name="velocity"/>
+                <command_interface name="position"/>
+                <command_interface name="la_reset"/>
+                <state_interface name="position"/>
+                <state_interface name="velocity"/>
+            </joint>
+            <joint name="Excavation_Rotate">
+                <command_interface name="velocity">
+                    <param name="min">-10</param>
+                    <param name="max">10</param>
+                </command_interface>
+                <command_interface name="position"/>
+                <state_interface name="position"/>
+                <state_interface name="velocity"/>
+            </joint>
+            <!-- <gpio name="vibe_control">
+                <command_interface name="vibe_enabled"/>
+            </gpio>
+            <gpio name="latch_control">
+                <command_interface name="hop_latched"/>
+            </gpio> -->
         </ros2_control>
-        <gazebo>
-            <plugin name="gz_ros2_control::GazeboSimROS2ControlPlugin" filename="libgz_ros2_control-system.so">
-                <parameters>$(find control)/config/tibble_controller.yaml</parameters>
-            </plugin>
-        </gazebo>
     </xacro:if>
 </robot>

File: src/description/urdf/sensors.xacro (robot description, xacro)
@@ -1,4 +1,53 @@
 <?xml version="1.0" encoding="utf-8"?>
 <robot xmlns:xacro="http://www.ros.org/wiki/xacro">
-    <!-- Define the joint/link for the sensors -->
+  <!-- 2D LiDAR -->
+  <joint name="lidar_joint" type="fixed">
+    <parent link="chassis_link" />
+    <child link="lidar_link" />
+    <origin xyz="0 0 0.1" rpy="0 0 0" />
+  </joint>
+  <link name="lidar_link">
+    <visual>
+      <geometry>
+        <cylinder length="0.05" radius="0.05" />
+      </geometry>
+      <material name="red" />
+    </visual>
+    <collision>
+      <geometry>
+        <cylinder length="0.05" radius="0.05" />
+      </geometry>
+    </collision>
+  </link>
+  <joint name="lidar_optical_joint" type="fixed">
+    <parent link="lidar_link" />
+    <child link="lidar_link_optical" />
+    <origin xyz="0.05 0 0" rpy="0 0 0" />
+  </joint>
+  <link name="lidar_link_optical"></link>
+  <!-- RGBD Camera -->
+  <joint name="camera_joint" type="fixed">
+    <parent link="chassis_link" />
+    <child link="camera_link" />
+    <origin xyz="0.205 0 0" rpy="0 0 0" />
+  </joint>
+  <link name="camera_link">
+    <visual>
+      <geometry>
+        <box size="0.010 0.03 0.03" />
+      </geometry>
+      <material name="orange" />
+    </visual>
+    <collision>
+      <geometry>
+        <box size="0.010 0.03 0.03"/>
+      </geometry>
+    </collision>
+  </link>
+  <joint name="camera_optical_joint" type="fixed">
+    <parent link="camera_link" />
+    <child link="camera_link_optical" />
+    <origin xyz="0 0 0" rpy="${-pi/2} 0 ${-pi/2}" />
+  </joint>
+  <link name="camera_link_optical"></link>
 </robot>

File: src/description/urdf/tibble.urdf.xacro (robot description, xacro)
@@ -14,5 +14,5 @@
     </xacro:if>
     <xacro:if value="$(arg use_sim)">
-        <xacro:include filename="gazebo.xacro"/>
+        <xacro:include filename="mujoco_inputs.xacro"/>
     </xacro:if>
 </robot>

Commit message: Replace Gazebo ros2_control with mujoco_ros2 control

File: src/description/urdf/ros2_control.xacro (robot description, xacro)
@@ -60,15 +60,50 @@
     <!-- Load the ROS2 Control information for just sim purposes -->
     <xacro:if value="$(arg use_sim)">
-        <ros2_control name="name" type="system">
+        <ros2_control name="MujocoSystem" type="system">
             <hardware>
-                <plugin>gz_ros2_control/GazeboSimSystem</plugin>
+                <plugin>mujoco_ros2_control/MujocoSystemInterface</plugin>
+                <param name="pids_config_file">$(find sim)/config/mujoco_pids.yaml</param>
             </hardware>
-            <!-- Define all joints and their command/state interfaces necessary for sim -->
+            <!-- Define all the joints that will have a command or state interface -->
+            <joint name="DL_Rotate">
+                <command_interface name="velocity">
+                    <param name="min">-10</param>
+                    <param name="max">10</param>
+                </command_interface>
+                <command_interface name="position"/>
+                <state_interface name="position"/>
+                <state_interface name="velocity"/>
+            </joint>
+            <joint name="DR_Rotate">
+                <command_interface name="velocity">
+                    <param name="min">-10</param>
+                    <param name="max">10</param>
+                </command_interface>
+                <command_interface name="position"/>
+                <state_interface name="position"/>
+                <state_interface name="velocity"/>
+            </joint>
+            <joint name="LA_Extend">
+                <command_interface name="velocity"/>
+                <command_interface name="position"/>
+                <state_interface name="position"/>
+                <state_interface name="velocity"/>
+            </joint>
+            <joint name="Excavation_Rotate">
+                <command_interface name="velocity">
+                    <param name="min">-10</param>
+                    <param name="max">10</param>
+                </command_interface>
+                <command_interface name="position"/>
+                <state_interface name="position"/>
+                <state_interface name="velocity"/>
+            </joint>
+            <!-- <gpio name="vibe_control">
+                <command_interface name="vibe_enabled"/>
+            </gpio>
+            <gpio name="latch_control">
+                <command_interface name="hop_latched"/>
+            </gpio> -->
         </ros2_control>
-        <gazebo>
-            <plugin name="gz_ros2_control::GazeboSimROS2ControlPlugin" filename="libgz_ros2_control-system.so">
-                <parameters>$(find control)/config/tibble_controller.yaml</parameters>
-            </plugin>
-        </gazebo>
     </xacro:if>
 </robot>

Commit message: Fix joints not being published by MuJoCo

File: src/description/urdf/ros2_control.xacro (robot description, xacro)
@@ -99,4 +99,61 @@
                 <state_interface name="velocity"/>
             </joint>
+            <!-- Joints that don't need control still need state_interface for MuJoCo -->
+            <joint name="DL_Rotate">
+                <state_interface name="position"/>
+                <state_interface name="velocity"/>
+            </joint>
+            <joint name="DR_Rotate">
+                <state_interface name="position"/>
+                <state_interface name="velocity"/>
+            </joint>
+            <joint name="DL_Rotate">
+                <state_interface name="position"/>
+                <state_interface name="velocity"/>
+            </joint>
+            <joint name="LLA_Rotate">
+                <state_interface name="position"/>
+                <state_interface name="velocity"/>
+            </joint>
+            <joint name="TLA_Rotate">
+                <state_interface name="position"/>
+                <state_interface name="velocity"/>
+            </joint>
+            <joint name="Hopper_Rotate">
+                <state_interface name="position"/>
+                <state_interface name="velocity"/>
+            </joint>
+            <joint name="HopperDoorRotate">
+                <state_interface name="position"/>
+                <state_interface name="velocity"/>
+            </joint>
+            <joint name="H-Latch_Rotate">
+                <state_interface name="position"/>
+                <state_interface name="velocity"/>
+            </joint>
+            <joint name="ML_Wheel_Rotate">
+                <state_interface name="position"/>
+                <state_interface name="velocity"/>
+            </joint>
+            <joint name="MR_Wheel_Rotate">
+                <state_interface name="position"/>
+                <state_interface name="velocity"/>
+            </joint>
+            <joint name="BL_Wheel_Rotate">
+                <state_interface name="position"/>
+                <state_interface name="velocity"/>
+            </joint>
+            <joint name="BR_Wheel_Rotate">
+                <state_interface name="position"/>
+                <state_interface name="velocity"/>
+            </joint>
+            <joint name="TL_Wheel_Rotate">
+                <state_interface name="position"/>
+                <state_interface name="velocity"/>
+            </joint>
+            <joint name="TR_Wheel_Rotate">
+                <state_interface name="position"/>
+                <state_interface name="velocity"/>
+            </joint>
             <!-- <gpio name="vibe_control">
                 <command_interface name="vibe_enabled"/>
