Commit message: Add back dummy sensors with updated positions

File: src/description/urdf/sensors.xacro (robot description, xacro)
@@ -1,4 +1,51 @@
 <?xml version="1.0" encoding="utf-8"?>
 <robot xmlns:xacro="http://www.ros.org/wiki/xacro">
-    <!-- Define the joint/link for the sensors -->
+  <!-- 2D LiDAR -->
+  <joint name="lidar_joint" type="fixed">
+    <parent link="chassis_link" />
+    <child link="lidar_link" />
+    <origin xyz="0.6 -1.91 1.25" rpy="${pi/2} 0 0" />
+  </joint>
+  <link name="lidar_link">
+    <visual>
+      <geometry>
+        <cylinder length="0.05" radius="0.05" />
+      </geometry>
+    </visual>
+    <collision>
+      <geometry>
+        <cylinder length="0.05" radius="0.05" />
+      </geometry>
+    </collision>
+  </link>
+  <joint name="lidar_optical_joint" type="fixed">
+    <parent link="lidar_link" />
+    <child link="lidar_link_optical" />
+    <origin xyz="0.05 0 0" rpy="0 0 0" />
+  </joint>
+  <link name="lidar_link_optical"></link>
+  <!-- RGBD Camera -->
+  <joint name="camera_joint" type="fixed">
+    <parent link="chassis_link" />
+    <child link="camera_link" />
+    <origin xyz="1.25 -1.65 1.25" rpy="0 0 ${pi/12}" />
+  </joint>
+  <link name="camera_link">
+    <visual>
+      <geometry>
+        <box size="0.010 0.03 0.03" />
+      </geometry>
+    </visual>
+    <collision>
+      <geometry>
+        <box size="0.010 0.03 0.03"/>
+      </geometry>
+    </collision>
+  </link>
+  <joint name="camera_optical_joint" type="fixed">
+    <parent link="camera_link" />
+    <child link="camera_link_optical" />
+    <origin xyz="0 0 0" rpy="${-pi/2} 0 ${-pi/2}" />
+  </joint>
+  <link name="camera_link_optical"></link>
 </robot>

Commit message: fixed the camera joint rotation so it properly renders in rerun

File: src/description/urdf/sensors.xacro (robot description, xacro)
@@ -29,5 +29,5 @@
     <parent link="chassis_link" />
     <child link="camera_link" />
-    <origin xyz="1.25 -1.65 1.25" rpy="0 0 ${pi/12}" />
+    <origin xyz="1.25 -1.65 1.25" rpy="${pi/2} 0 ${pi/12}" />
   </joint>
   <link name="camera_link">
